File: example-E.kicad_sch (KiCad schematic)
At the start: 21 parts

Commit message: Finished story
Connections:
- net BAT_SW: now also U304.1 (OUT), U307.5 (VCC), U309.5 (VCC)
- net EN_Out: now also U309.4
- net VBat_In: now also U304.4 (IN)
- net ~{Activate}: now also U307.2
- net ~{KFC1}: now also Q301.1
- net ~{RBF_PIN1}: now also U304.3 (ON)
- new net: Q301.2, U309.6
- new net: U304.2 (GND), U304.5 (GND)
