File: example-NE.kicad_sch (KiCad schematic)
At the start: 0 parts

Commit message: Finished story
Parts:
- added C302, C304, C305, C307, C310, C312, C314, C315: (no value), symbol Device:C
- added F301: (no value), symbol Device:Fuse
- added Q301: (no value), symbol lsf-kicad:FDN537N
- added R306, R314, R315, R316, R317, R318, R319, R321: (no value), symbol Device:R
- added U304: (no value), symbol Power_Management:SiP32431DR3
- added U307: (no value), symbol 74xGxx:74AHC1G04
- added U309: (no value), symbol 74xGxx:74LVC1G332
Connections:
- new net: F301.1, R317.2
- new net: C314.1, R318.1
- new net: C315.1, R319.1
- new net BAT_SW: C302.1, C304.1, C305.1, C310.1, R314.1, R316.1, R317.1
- new net EN_Out: R315.1, R319.2, R321.2
- new net VBat_In: C307.1, R306.1
- new net ~{Activate}: R314.2
- new net ~{KFC1}: C312.1, R315.2
- new net ~{RBF_PIN1}: R306.2
