File: activator-prsd.kicad_sch (KiCad schematic)
At the start: 21 parts, among them Q301 FDN337N, U304 SiP32431DR3, U307 74AHC1G04, U309 74LVC1G332

Commit message: ocr fix :)
Connections:
- net BAT_SW: no longer U304.1 (OUT), U307.5 (VCC), U309.5 (VCC)
- net EN_Out: no longer U309.4
- net VBat_In: no longer U304.4 (IN)
- net ~{Activate}: no longer U307.2
- net ~{RBF_PIN1}: no longer U304.3 (ON)
- net at Q301.2: no longer U309.6

Commit message: changed back to old ocr
Connections:
- net BAT_SW: now also U304.1 (OUT), U307.5 (VCC), U309.5 (VCC)
- net EN_Out: now also U309.4
- net VBat_In: now also U304.4 (IN)
- net ~{Activate}: now also U307.2
- net ~{RBF_PIN1}: now also U304.3 (ON)
- net at Q301.2: now also U309.6
- new net: U304.2 (GND), U304.5 (GND)
