File: activator-prsd.kicad_sch (KiCad schematic)
At the start: 21 parts, among them Q301 FDN337N, U304 SiP32431DR3, U307 74AHC1G04, U309 74LVC1G332

Commit message: draft done
Connections:
- net BAT_SW: no longer U304.1 (OUT)
- net VBat_In: no longer U304.4 (IN)
- net ~{KFC1}: no longer Q301.1
- net ~{RBF_PIN1}: no longer U304.3 (ON)
- net at U309.6: no longer Q301.2
