File: result.kicad_sch (KiCad schematic)
At the start: 68 parts, among them Q801 FDN308P, U801 BD226xG-M, U802 SKYA21003, U803 PAT0816-C-10DB, U804 QPA4263C, U805 RF1419D, U806 74AUP2G14, U808 RF1419D, U810 TQP3M9036, U811 TSV7723, U812 BGA6130, U813 LTC5507ES6PBF, U814 LTC5507ES6PBF, U815 LFCG-490+, U816 SKYA21003

Commit message: merging to main
Parts:
- removed C801, C809, C812: 1uF, Capacitor_SMD:C_0402_1005Metric, symbol Device:C
- removed C802, C804, C823, C824, C825, C826: 220pF, Capacitor_SMD:C_0402_1005Metric, symbol Device:C
- removed C803: 0 Ohm, Capacitor_SMD:C_0402_1005Metric, symbol Device:C
- removed C805, C808, C810, C817: 100pF, Capacitor_SMD:C_0402_1005Metric, symbol Device:C
- removed C806: 20pF, Capacitor_SMD:C_0402_1005Metric, symbol Device:C
- removed C807: 15pF, Capacitor_SMD:C_0402_1005Metric, symbol Device:C
- removed C811, C820, C827: 1nF, Capacitor_SMD:C_0402_1005Metric, symbol Device:C
- removed C815: 47nF, Capacitor_SMD:C_0402_1005Metric, symbol Device:C
- removed C816: 2.36pF, Capacitor_SMD:C_0402_1005Metric, symbol Device:C
- removed C818: 10uF, Capacitor_SMD:C_0402_1005Metric, symbol Device:C
- removed C819: 100nF, Capacitor_SMD:C_0402_1005Metric, symbol Device:C
- removed C821: Open, Capacitor_SMD:C_0402_1005Metric, symbol Device:C
- removed C822: 18pF, Capacitor_SMD:C_0402_1005Metric, symbol Device:C
- removed C828, C829: 10pF, Capacitor_SMD:C_0402_1005Metric, symbol Device:C
- removed L801, L806: 68nH, Inductor_SMD:L_0402_1005Metric, symbol Device:L
- removed L802: 18nH, Inductor_SMD:L_0402_1005Metric, symbol Device:L
- removed L809: 8.2nH, Inductor_SMD:L_0402_1005Metric, symbol Device:L
- removed L810: 68nH, Inductor_SMD:L_0603_1608Metric, symbol Device:L
- removed L811: 43 nH, Inductor_SMD:L_0402_1005Metric, symbol Device:L
- removed Q801: FDN308P, Package_TO_SOT_SMD:SOT-23, symbol Transistor_FET:FDN340P
- removed R801: 100k, Resistor_SMD:R_0402_1005Metric, symbol Device:R
- removed R802: 1k, Resistor_SMD:R_0402_1005Metric, symbol Device:R
- removed R803, R804, R810, R811, R813, R815, R817: 10k, Resistor_SMD:R_0402_1005Metric, symbol Device:R
- removed R805: 120, Resistor_SMD:R_0402_1005Metric, symbol Device:R
- removed R808: 270, Resistor_SMD:R_0402_1005Metric, symbol Device:R
- removed R809: 3k9, Resistor_SMD:R_0402_1005Metric, symbol Device:R
- removed R812: 33k, Resistor_SMD:R_0402_1005Metric, symbol Device:R
- removed R814, R816: 2k7, Resistor_SMD:R_0402_1005Metric, symbol Device:R
- removed R818: 453, Resistor_SMD:R_0402_1005Metric, symbol Device:R
- removed R819: 54.9, Resistor_SMD:R_0402_1005Metric, symbol Device:R
- removed RN801, RN802: 4.7k, Resistor_SMD:R_Array_Convex_4x0402, symbol Device:R_Pack04
- removed TP801: MS-156C3, lsf-kicad-lib:MS-156C3, symbol lsf-kicad:MS-156C3
- removed U801: BD226xG-M, lsf-kicad-lib:ROHM_SSOP-5, symbol lsf-kicad:BD226xG-M
- removed U802, U816: SKYA21003, lsf-kicad-lib:QFN-12-1EP_2x2mm_P0.5mm_EP0.76x0.76mm, symbol lsf-kicad:SKYA21003
- removed U803: PAT0816-C-10DB, lsf-kicad-lib:RF_Attenuator_Susumu_PAT0816, symbol RF:PAT1220-C-5DB
- removed U804: QPA4263C, Package_TO_SOT_SMD:SOT-363_SC-70-6, symbol lsf-kicad:QPA4263C
- removed U805, U808: RF1419D, lsf-kicad-lib:SM3838-8, symbol lsf-kicad:RF1419D
- removed U806: 74AUP2G14, Package_TO_SOT_SMD:SOT-363_SC-70-6, symbol lsf-kicad:74AUP2G14
- removed U810: TQP3M9036, lsf-kicad-lib:DFN-8-1EP_2x2mm_P0.5mm_EP0.7x1.6mm_ThermalVias, symbol lsf-kicad:TQP3M9036
- removed U811: TSV7723, Package_SO:MSOP-10_3x3mm_P0.5mm, symbol lsf-kicad:TSV7723
- removed U812: BGA6130, lsf-kicad-lib:NXP_HVSON-8, symbol lsf-kicad:BGA6130
- removed U813, U814: LTC5507ES6PBF, Package_TO_SOT_SMD:TSOT-23-6, symbol lsf-kicad:LTC5507
- removed U815: LFCG-490+, lsf-kicad-lib:GE0805C-2, symbol lsf-kicad:LFCG-490+
- added H1, H2, H3, H4: MountingHole, MountingHole:MountingHole_3.2mm_M3_DIN965_Pad, symbol Mechanical:MountingHole
- added JP1, JP2, JP3, JP4: SolderJumper_3_Bridged12, Jumper:SolderJumper-3_P1.3mm_Bridged12_RoundedPad1.0x1.5mm_NumberLabels, symbol Jumper:SolderJumper_3_Bridged12
- added JP5, JP6: SolderJumper_2_Open, Jumper:SolderJumper-2_P1.3mm_Open_RoundedPad1.0x1.5mm, symbol Jumper:SolderJumper_2_Open
- added LOGO1, LOGO3: nush_logo, cubesat_obc:nush, symbol cubesat_obc_lib:nush_logo
- added LOGO2, LOGO4: galileo_logo, cubesat_obc:logo, symbol cubesat_obc_lib:galileo_logo
- added LOGO5: axes_logo, cubesat_obc:axes, symbol cubesat_obc_lib:axes_logo
- added LOGO6: axes_logo_inv, cubesat_obc:axes_inv, symbol cubesat_obc_lib:axes_logo
- added R1: 39k, Resistor_SMD:R_0402_1005Metric, symbol Device:R
- added R2: 20k, Resistor_SMD:R_0603_1608Metric, symbol Device:R
- added SPI1, UART_1, UART_OBC_1: Conn_01x05_Female, Connector_Molex:Molex_PicoBlade_53261-0571_1x05-1MP_P1.25mm_Horizontal, symbol Connector_Generic_MountingPin:Conn_01x05_MountingPin
- added UART_FTDI1: Conn_01x08_Female, Connector_Molex:Molex_PicoBlade_53261-0871_1x08-1MP_P1.25mm_Horizontal, symbol Connector_Generic_MountingPin:Conn_01x08_MountingPin
Connections:
- new net 3V3_3: UART_FTDI1.2 (Pin_2)
- new net CS3: SPI1.5 (Pin_5)
- new net GND: R2.2, SPI1.1 (Pin_1), SPI1.MP (MountPin), UART_1.1 (Pin_1), UART_1.MP (MountPin), UART_FTDI1.1 (Pin_1), UART_FTDI1.MP (MountPin), UART_OBC_1.1 (Pin_1), UART_OBC_1.MP (MountPin)
- new net MISO_2: SPI1.2 (Pin_2)
- new net MOSI_2: SPI1.3 (Pin_3)
- new net RX1_FTDI: JP3.1 (A), UART_FTDI1.4 (Pin_4)
- new net RX1_OBC: JP3.3 (B), UART_OBC_1.3 (Pin_3)
- new net RX2_FTDI: JP4.1 (A), UART_FTDI1.6 (Pin_6)
- new net RX2_OBC: JP4.3 (B), UART_OBC_1.5 (Pin_5)
- new net RX3_FTDI: JP6.1 (A), UART_FTDI1.8 (Pin_8)
- new net RX3_OBC: JP6.2 (B)
- new net SCK_2: SPI1.4 (Pin_4)
- new net TX1_FTDI: JP1.1 (A), UART_FTDI1.3 (Pin_3)
- new net TX1_OBC: JP1.3 (B), UART_OBC_1.2 (Pin_2)
- new net TX2_FTDI: JP2.1 (A), UART_FTDI1.5 (Pin_5)
- new net TX2_OBC: JP2.3 (B), UART_OBC_1.4 (Pin_4)
- new net TX3_FTDI: JP5.1 (A), UART_FTDI1.7 (Pin_7)
- new net TX3_OBC: JP5.2 (B)
- new net UART1_RX: UART_1.3 (Pin_3)
- new net UART1_TX: UART_1.2 (Pin_2)
- new net UART3_RX: UART_1.5 (Pin_5)
- new net UART3_TX: UART_1.4 (Pin_4)
- new net VBAT: R1.1
- new net mcu/ADC12_IN15: R1.2, R2.1
- new net modules/UART0_RX: JP1.2 (C)
- new net modules/UART0_TX: JP3.2 (C)
- new net modules/UART2_RX: JP2.2 (C)
- new net modules/UART2_TX: JP4.2 (C)
- no-connect marks 1 -> 2
Other:
- added sheet ftdi (ftdi.kicad_sch)
- added sheet imu_gps (imu_gps.kicad_sch)
- added sheet magnetorquer (magnetorquer.kicad_sch)
- added sheet mcu (mcu.kicad_sch)
- added sheet memory (memory.kicad_sch)
- added sheet modules (modules.kicad_sch)
- added sheet photodiode_preamps (photodiode_preamps.kicad_sch)
- added sheet stacking_connector (stacking_connector.kicad_sch)
- added sheet temp_sensors (temp_sensors.kicad_sch)
- note removed: "+5.4dBm to + 26.0dBm"
- note removed: "-10dBm to +15dBm"
- note removed: "-23dBm to +2dBm"
- note removed: "-9.1dBm to + 14.3dBm"
- note removed: "RF1419D IL 1.6 dB Fc = 403.5 BW = 7.5 MHz This is placed after the 1st LNA to improve Detectivity"
- note removed: "RF1419D This is placed before the HPA since it cannot handle the power Rated for 10dBm"
- note removed: "RX Chain Power ON: TQP3M9036 -> 45mA Power STNDBY: TQP3M9036 -> 4mA Switching speeds: TQP3M9036 -> 1us Totals: ON state: < 45mA max OFF state: < 20uA Switch ON speed: 1 usec Switch OFF speed: 1 usec"
- note removed: "TQP3M9036 NF = 0.45 Can be replaced by GRF2070 (NF=0.35) with small changes"
- note removed: "TX Chain Power ON (no RF): 1x BGA6130 -> 71mA 1x QPA4263C-> 55mA 2x LTC5507 -> 1.7mA 2x TSV7723 -> 5mA Power ON (RF): 1x BGA6130 -> 200mA 1x QPA4263C-> 55mA 2x LTC5507 -> 1.7mA 2x TSV7723 -> 5mA Power STNDBY: 1x BGA6130 -> 6uA 1x QPA4263C-> 0mA 2x LTC5507 -> 8uA 2x TSV7723 -> 16uA Switching speeds: 1x BGA6130 -> 2.2us(PWRUP), 0.5us(PWRDN) 1x QPA4263C-> To be measured 2x LTC5507 -> 7-20us 2x TSV77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"
- note removed: "The R divider ensures Ven<3V Making the board 5V compliant"
- note removed: "The resistive tap is -25dB to ensure: * Dynamic range match to LTC5507 * Minimal power loss to main signal"
- note removed: "This is needed to stop Tx_EN High during PWR_DN mode"
- title: (none) -> CubeSat On Board Computer

Commit message: fixed component selection
Parts:
- removed H1, H2, H3, H4: MountingHole, MountingHole:MountingHole_3.2mm_M3_DIN965_Pad, symbol Mechanical:MountingHole
- removed JP1, JP2, JP3, JP4: SolderJumper_3_Bridged12, Jumper:SolderJumper-3_P1.3mm_Bridged12_RoundedPad1.0x1.5mm_NumberLabels, symbol Jumper:SolderJumper_3_Bridged12
- removed JP5, JP6: SolderJumper_2_Open, Jumper:SolderJumper-2_P1.3mm_Open_RoundedPad1.0x1.5mm, symbol Jumper:SolderJumper_2_Open
- removed LOGO1, LOGO3: nush_logo, cubesat_obc:nush, symbol cubesat_obc_lib:nush_logo
- removed LOGO2, LOGO4: galileo_logo, cubesat_obc:logo, symbol cubesat_obc_lib:galileo_logo
- removed LOGO5: axes_logo, cubesat_obc:axes, symbol cubesat_obc_lib:axes_logo
- removed LOGO6: axes_logo_inv, cubesat_obc:axes_inv, symbol cubesat_obc_lib:axes_logo
- removed R1: 39k, Resistor_SMD:R_0402_1005Metric, symbol Device:R
- removed R2: 20k, Resistor_SMD:R_0603_1608Metric, symbol Device:R
- removed SPI1, UART_1, UART_OBC_1: Conn_01x05_Female, Connector_Molex:Molex_PicoBlade_53261-0571_1x05-1MP_P1.25mm_Horizontal, symbol Connector_Generic_MountingPin:Conn_01x05_MountingPin
- removed UART_FTDI1: Conn_01x08_Female, Connector_Molex:Molex_PicoBlade_53261-0871_1x08-1MP_P1.25mm_Horizontal, symbol Connector_Generic_MountingPin:Conn_01x08_MountingPin
- added C801, C809, C812: 1uF, Capacitor_SMD:C_0402_1005Metric, symbol Device:C
- added C802, C804, C823, C824, C825, C826: 220pF, Capacitor_SMD:C_0402_1005Metric, symbol Device:C
- added C803: 0 Ohm, Capacitor_SMD:C_0402_1005Metric, symbol Device:C
- added C805, C808, C810, C817: 100pF, Capacitor_SMD:C_0402_1005Metric, symbol Device:C
- added C806: 20pF, Capacitor_SMD:C_0402_1005Metric, symbol Device:C
- added C807: 15pF, Capacitor_SMD:C_0402_1005Metric, symbol Device:C
- added C811, C820, C827: 1nF, Capacitor_SMD:C_0402_1005Metric, symbol Device:C
- added C815: 47nF, Capacitor_SMD:C_0402_1005Metric, symbol Device:C
- added C816: 2.36pF, Capacitor_SMD:C_0402_1005Metric, symbol Device:C
- added C818: 10uF, Capacitor_SMD:C_0402_1005Metric, symbol Device:C
- added C819: 100nF, Capacitor_SMD:C_0402_1005Metric, symbol Device:C
- added C821: Open, Capacitor_SMD:C_0402_1005Metric, symbol Device:C
- added C822: 18pF, Capacitor_SMD:C_0402_1005Metric, symbol Device:C
- added C828, C829: 10pF, Capacitor_SMD:C_0402_1005Metric, symbol Device:C
- added L801, L806: 68nH, Inductor_SMD:L_0402_1005Metric, symbol Device:L
- added L802: 18nH, Inductor_SMD:L_0402_1005Metric, symbol Device:L
- added L809: 8.2nH, Inductor_SMD:L_0402_1005Metric, symbol Device:L
- added L810: 68nH, Inductor_SMD:L_0603_1608Metric, symbol Device:L
- added L811: 43 nH, Inductor_SMD:L_0402_1005Metric, symbol Device:L
- added Q801: FDN308P, Package_TO_SOT_SMD:SOT-23, symbol Transistor_FET:FDN340P
- added R801: 100k, Resistor_SMD:R_0402_1005Metric, symbol Device:R
- added R802: 1k, Resistor_SMD:R_0402_1005Metric, symbol Device:R
- added R803, R804, R810, R811, R813, R815, R817: 10k, Resistor_SMD:R_0402_1005Metric, symbol Device:R
- added R805: 120, Resistor_SMD:R_0402_1005Metric, symbol Device:R
- added R808: 270, Resistor_SMD:R_0402_1005Metric, symbol Device:R
- added R809: 3k9, Resistor_SMD:R_0402_1005Metric, symbol Device:R
- added R812: 33k, Resistor_SMD:R_0402_1005Metric, symbol Device:R
- added R814, R816: 2k7, Resistor_SMD:R_0402_1005Metric, symbol Device:R
- added R818: 453, Resistor_SMD:R_0402_1005Metric, symbol Device:R
- added R819: 54.9, Resistor_SMD:R_0402_1005Metric, symbol Device:R
- added RN801, RN802: 4.7k, Resistor_SMD:R_Array_Convex_4x0402, symbol Device:R_Pack04
- added TP801: MS-156C3, lsf-kicad-lib:MS-156C3, symbol lsf-kicad:MS-156C3
- added U801: BD226xG-M, lsf-kicad-lib:ROHM_SSOP-5, symbol lsf-kicad:BD226xG-M
- added U802, U816: SKYA21003, lsf-kicad-lib:QFN-12-1EP_2x2mm_P0.5mm_EP0.76x0.76mm, symbol lsf-kicad:SKYA21003
- added U803: PAT0816-C-10DB, lsf-kicad-lib:RF_Attenuator_Susumu_PAT0816, symbol RF:PAT1220-C-5DB
- added U804: QPA4263C, Package_TO_SOT_SMD:SOT-363_SC-70-6, symbol lsf-kicad:QPA4263C
- added U805, U808: RF1419D, lsf-kicad-lib:SM3838-8, symbol lsf-kicad:RF1419D
- added U806: 74AUP2G14, Package_TO_SOT_SMD:SOT-363_SC-70-6, symbol lsf-kicad:74AUP2G14
- added U810: TQP3M9036, lsf-kicad-lib:DFN-8-1EP_2x2mm_P0.5mm_EP0.7x1.6mm_ThermalVias, symbol lsf-kicad:TQP3M9036
- added U811: TSV7723, Package_SO:MSOP-10_3x3mm_P0.5mm, symbol lsf-kicad:TSV7723
- added U812: BGA6130, lsf-kicad-lib:NXP_HVSON-8, symbol lsf-kicad:BGA6130
- added U813, U814: LTC5507ES6PBF, Package_TO_SOT_SMD:TSOT-23-6, symbol lsf-kicad:LTC5507
- added U815: LFCG-490+, lsf-kicad-lib:GE0805C-2, symbol lsf-kicad:LFCG-490+
Connections:
- new net: R817.1, U811.7 (+), U814.3 (VOUT)
- new net: R811.2, R816.1, U811.8 (-)
- new net: R810.2, R814.1, U811.2 (-)
- new net: C827.1, U815.8 (IN)
- new net: C821.2, C822.2, C827.2, L809.2, L810.1
- new net: L809.1, U812.2 (RF_OUT), U812.3 (RF_OUT)
- new net: C823.1, C828.1, L811.1, R818.2, R819.1
- new net: C805.2, C811.2, C812.2, L801.2, Q801.3 (D)
- new net: R818.1, TP801.C
- new net: C803.1, C806.2, L802.1
- new net: C803.2, C804.1
- new net: C807.2, L802.2, R805.1
- new net: C807.1, R805.2, U812.7 (RF_IN)
- new net: C808.1, U808.2 (IN)
- new net: R808.1, U812.6 (EN)
- new net: C808.2, L806.1, U810.7 (RFOUT)
- new net: C823.2, U813.6 (RF_IN)
- new net: C816.1, C817.1, U810.2 (RFIN)
- new net: C804.2, L801.1, U804.6 (RFOUT)
- new net: C802.1, U804.3 (RFIN)
- new net: C802.2, U805.6 (OUT)
- new net: C826.1, U814.5 (PCAP)
- new net: C825.2, U814.6 (RF_IN)
- new net: C825.1, C829.1, L811.2
- new net: Q801.1 (G), R801.2, R802.1
- new net: R809.1, U812.8 (ICQ_ADJ)
- new net: RN802.3 (R3.1), RN802.4 (R4.1), U816.7 (CTRL)
- new net: RN802.1 (R1.1), RN802.2 (R2.1), U816.8 (EN)
- new net: RN801.1 (R1.1), RN801.2 (R2.1), U802.7 (CTRL)
- new net: RN801.3 (R3.1), RN801.4 (R4.1), U802.8 (EN)
- new net: R812.1, R813.2, U810.6 (Shut_Down)
- new net: R815.1, U811.3 (+), U813.3 (VOUT)
- new net: U803.2, U805.2 (IN)
- new net: C824.2, U813.5 (PCAP)
- new net 3V3: C801.1, U801.1 (IN)
- new net ANT: U816.2 (RF1)
- new net EN: R803.2, U801.3 (EN)
- new net FSENSE: R811.1, U811.9
- new net GNDA: C801.2, C805.1, C806.1, C809.2, C810.2, C811.1, C812.1, C815.2, C816.2, C818.2, C819.2, C820.2, C821.1, C822.1, C828.2, C829.2, R803.1, R804.1, R809.2, R813.1, R814.2, R815.2, R816.2, R817.2, R819.2, RN801.6 (R3.2), RN801.8 (R1.2), RN802.6 (R3.2), RN802.8 (R1.2), TP801.G, U801.2 (GND), U802.1 (GND), U802.10 (GND), U802.12 (GND), U802.13 (EP), U802.3 (GND), U802.4 (GND), U802.6 (GND), U803.3, U804.1 (GND), U804.2 (GND), U804.4 (GND), U804.5 (GND), U805.1 (GND), U805.3 (GND), U805.4 (GND), U805.5 (GND), U805.7 (GND), U805.8 (GND), U806.2 (GND), U808.1 (GND), U808.3 (GND), U808.4 (GND), U808.5 (GND), U808.7 (GND), U808.8 (GND), U810.1 (NIC), U810.3 (NIC), U810.4 (NIC), U810.5 (NIC), U810.8 (NIC), U810.9 (GND), U811.4 (VCC-), U812.1 (NIC), U812.4 (NIC), U812.9 (EP_GND), U813.2 (GND), U814.2 (GND), U815.1 (GND), U815.2 (GND), U815.3 (GND), U815.5 (GND), U815.6 (GND), U815.7 (GND), U816.1 (GND), U816.10 (GND), U816.12 (GND), U816.13 (EP), U816.3 (GND), U816.4 (GND), U816.6 (GND)
- new net PSENSE: R810.1, U811.1
- new net RFFE_3V3: C809.1, C810.1, C815.1, C818.1, C819.1, C820.1, C824.1, C826.2, L806.2, L810.2, Q801.2 (S), R801.1, RN801.5 (R4.2), RN802.7 (R2.2), U801.5 (OUT), U802.9 (VCC), U806.5 (VCC), U811.10 (VCC+), U812.5 (VCC), U813.4 (VCC), U814.4 (VCC), U816.9 (VCC)
- new net RFIO: U802.2 (RF1)
- new net RX_RF_IN: C817.2, U816.5 (RF3)
- new net RX_RF_OUT: U802.5 (RF3), U808.6 (OUT)
- new net TX_EN: R804.2, U806.1
- new net TX_RF_IN: U802.11 (RF2), U803.1
- new net TX_RF_OUT: TP801.A, U815.4 (OUT), U816.11 (RF2)
- new net ~{ΤX_EN}: R802.2, U806.3, U806.6
- new net ΤX_EN_ΙΝΤ: R808.2, R812.2, RN801.7 (R2.2), RN802.5 (R4.2), U806.4, U811.5 (EN1), U811.6 (EN2), U813.1 (~{SHDN}), U814.1 (~{SHDN})
- no-connect marks 2 -> 1
Other:
- removed sheet ftdi
- removed sheet imu_gps
- removed sheet magnetorquer
- removed sheet mcu
- removed sheet memory
- removed sheet modules
- removed sheet photodiode_preamps
- removed sheet stacking_connector
- removed sheet temp_sensors
- note added: "+5.4dBm to + 26.0dBm"
- note added: "-10dBm to +15dBm"
- note added: "-23dBm to +2dBm"
- note added: "-9.1dBm to + 14.3dBm"
- note added: "RF1419D IL 1.6 dB Fc = 403.5 BW = 7.5 MHz This is placed after the 1st LNA to improve Detectivity"
- note added: "RF1419D This is placed before the HPA since it cannot handle the power Rated for 10dBm"
- note added: "RX Chain Power ON: TQP3M9036 -> 45mA Power STNDBY: TQP3M9036 -> 4mA Switching speeds: TQP3M9036 -> 1us Totals: ON state: < 45mA max OFF state: < 20uA Switch ON speed: 1 usec Switch OFF speed: 1 usec"
- note added: "TQP3M9036 NF = 0.45 Can be replaced by GRF2070 (NF=0.35) with small changes"
- note added: "TX Chain Power ON (no RF): 1x BGA6130 -> 71mA 1x QPA4263C-> 55mA 2x LTC5507 -> 1.7mA 2x TSV7723 -> 5mA Power ON (RF): 1x BGA6130 -> 200mA 1x QPA4263C-> 55mA 2x LTC5507 -> 1.7mA 2x TSV7723 -> 5mA Power STNDBY: 1x BGA6130 -> 6uA 1x QPA4263C-> 0mA 2x LTC5507 -> 8uA 2x TSV7723 -> 16uA Switching speeds: 1x BGA6130 -> 2.2us(PWRUP), 0.5us(PWRDN) 1x QPA4263C-> To be measured 2x LTC5507 -> 7-20us 2x TSV77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"
- note added: "The R divider ensures Ven<3V Making the board 5V compliant"
- note added: "The resistive tap is -25dB to ensure: * Dynamic range match to LTC5507 * Minimal power loss to main signal"
- note added: "This is needed to stop Tx_EN High during PWR_DN mode"
- title: CubeSat On Board Computer -> (none)
