File: result.kicad_sch (KiCad schematic)
At the start: 21 parts, among them Q301 FDN337N, U304 SiP32431DR3, U307 74AHC1G04, U309 74LVC1G332

Commit message: first draft, working on abstraction levels
Parts:
- removed C302, C304, C305, C310: 100nF, Capacitor_SMD:C_0402_1005Metric, symbol Device:C
- removed C307: 1uF, Capacitor_SMD:C_0402_1005Metric, symbol Device:C
- removed C312: 10uF, Capacitor_SMD:C_0402_1005Metric, symbol Device:C
- removed C314, C315: 22uF, Capacitor_SMD:C_0402_1005Metric, symbol Device:C
- removed F301: Fuse, Fuse:Fuse_0603_1608Metric, symbol Device:Fuse
- removed Q301: FDN337N, Package_TO_SOT_SMD:SuperSOT-3, symbol lsf-kicad:FDN537N
- removed R306: 1M, Resistor_SMD:R_0402_1005Metric, symbol Device:R
- removed R314, R317, R321: 100k, Resistor_SMD:R_0402_1005Metric, symbol Device:R
- removed R315, R318, R319: 10k, Resistor_SMD:R_0402_1005Metric, symbol Device:R
- removed R316: 10, Resistor_SMD:R_0402_1005Metric, symbol Device:R
- removed U304: SiP32431DR3, Package_TO_SOT_SMD:SOT-363_SC-70-6, symbol Power_Management:SiP32431DR3
- removed U307: 74AHC1G04, Package_TO_SOT_SMD:TSOT-23-5, symbol 74xGxx:74AHC1G04
- removed U309: 74LVC1G332, Package_TO_SOT_SMD:SOT-363_SC-70-6, symbol 74xGxx:74LVC1G332
- added C801, C809, C812: 1uF, Capacitor_SMD:C_0402_1005Metric, symbol Device:C
- added C802, C804, C823, C824, C825, C826: 220pF, Capacitor_SMD:C_0402_1005Metric, symbol Device:C
- added C803: 0 Ohm, Capacitor_SMD:C_0402_1005Metric, symbol Device:C
- added C805, C808, C810, C817: 100pF, Capacitor_SMD:C_0402_1005Metric, symbol Device:C
- added C806: 20pF, Capacitor_SMD:C_0402_1005Metric, symbol Device:C
- added C807: 15pF, Capacitor_SMD:C_0402_1005Metric, symbol Device:C
- added C811, C820, C827: 1nF, Capacitor_SMD:C_0402_1005Metric, symbol Device:C
- added C815: 47nF, Capacitor_SMD:C_0402_1005Metric, symbol Device:C
- added C816: 2.36pF, Capacitor_SMD:C_0402_1005Metric, symbol Device:C
- added C818: 10uF, Capacitor_SMD:C_0402_1005Metric, symbol Device:C
- added C819: 100nF, Capacitor_SMD:C_0402_1005Metric, symbol Device:C
- added C821: Open, Capacitor_SMD:C_0402_1005Metric, symbol Device:C
- added C822: 18pF, Capacitor_SMD:C_0402_1005Metric, symbol Device:C
- added C828, C829: 10pF, Capacitor_SMD:C_0402_1005Metric, symbol Device:C
- added L801, L806: 68nH, Inductor_SMD:L_0402_1005Metric, symbol Device:L
- added L802: 18nH, Inductor_SMD:L_0402_1005Metric, symbol Device:L
- added L809: 8.2nH, Inductor_SMD:L_0402_1005Metric, symbol Device:L
- added L810: 68nH, Inductor_SMD:L_0603_1608Metric, symbol Device:L
- added L811: 43 nH, Inductor_SMD:L_0402_1005Metric, symbol Device:L
- added Q801: FDN308P, Package_TO_SOT_SMD:SOT-23, symbol Transistor_FET:FDN340P
- added R801: 100k, Resistor_SMD:R_0402_1005Metric, symbol Device:R
- added R802: 1k, Resistor_SMD:R_0402_1005Metric, symbol Device:R
- added R803, R804, R810, R811, R813, R815, R817: 10k, Resistor_SMD:R_0402_1005Metric, symbol Device:R
- added R805: 120, Resistor_SMD:R_0402_1005Metric, symbol Device:R
- added R808: 270, Resistor_SMD:R_0402_1005Metric, symbol Device:R
- added R809: 3k9, Resistor_SMD:R_0402_1005Metric, symbol Device:R
- added R812: 33k, Resistor_SMD:R_0402_1005Metric, symbol Device:R
- added R814, R816: 2k7, Resistor_SMD:R_0402_1005Metric, symbol Device:R
- added R818: 453, Resistor_SMD:R_0402_1005Metric, symbol Device:R
- added R819: 54.9, Resistor_SMD:R_0402_1005Metric, symbol Device:R
- added RN801, RN802: 4.7k, Resistor_SMD:R_Array_Convex_4x0402, symbol Device:R_Pack04
- added TP801: MS-156C3, lsf-kicad-lib:MS-156C3, symbol lsf-kicad:MS-156C3
- added U801: BD226xG-M, lsf-kicad-lib:ROHM_SSOP-5, symbol lsf-kicad:BD226xG-M
- added U802, U816: SKYA21003, lsf-kicad-lib:QFN-12-1EP_2x2mm_P0.5mm_EP0.76x0.76mm, symbol lsf-kicad:SKYA21003
- added U803: PAT0816-C-10DB, lsf-kicad-lib:RF_Attenuator_Susumu_PAT0816, symbol RF:PAT1220-C-5DB
- added U804: QPA4263C, Package_TO_SOT_SMD:SOT-363_SC-70-6, symbol lsf-kicad:QPA4263C
- added U805, U808: RF1419D, lsf-kicad-lib:SM3838-8, symbol lsf-kicad:RF1419D
- added U806: 74AUP2G14, Package_TO_SOT_SMD:SOT-363_SC-70-6, symbol lsf-kicad:74AUP2G14
- added U810: TQP3M9036, lsf-kicad-lib:DFN-8-1EP_2x2mm_P0.5mm_EP0.7x1.6mm_ThermalVias, symbol lsf-kicad:TQP3M9036
- added U811: TSV7723, Package_SO:MSOP-10_3x3mm_P0.5mm, symbol lsf-kicad:TSV7723
- added U812: BGA6130, lsf-kicad-lib:NXP_HVSON-8, symbol lsf-kicad:BGA6130
- added U813, U814: LTC5507ES6PBF, Package_TO_SOT_SMD:TSOT-23-6, symbol lsf-kicad:LTC5507
- added U815: LFCG-490+, lsf-kicad-lib:GE0805C-2, symbol lsf-kicad:LFCG-490+
Connections:
- new net: R817.1, U811.7 (+), U814.3 (VOUT)
- new net: R811.2, R816.1, U811.8 (-)
- new net: R810.2, R814.1, U811.2 (-)
- new net: C827.1, U815.8 (IN)
- new net: C821.2, C822.2, C827.2, L809.2, L810.1
- new net: L809.1, U812.2 (RF_OUT), U812.3 (RF_OUT)
- new net: C823.1, C828.1, L811.1, R818.2, R819.1
- new net: C805.2, C811.2, C812.2, L801.2, Q801.3 (D)
- new net: R818.1, TP801.C
- new net: C803.1, C806.2, L802.1
- new net: C803.2, C804.1
- new net: C807.2, L802.2, R805.1
- new net: C807.1, R805.2, U812.7 (RF_IN)
- new net: C808.1, U808.2 (IN)
- new net: R808.1, U812.6 (EN)
- new net: C808.2, L806.1, U810.7 (RFOUT)
- new net: C823.2, U813.6 (RF_IN)
- new net: C816.1, C817.1, U810.2 (RFIN)
- new net: C804.2, L801.1, U804.6 (RFOUT)
- new net: C802.1, U804.3 (RFIN)
- new net: C802.2, U805.6 (OUT)
- new net: C826.1, U814.5 (PCAP)
- new net: C825.2, U814.6 (RF_IN)
- new net: C825.1, C829.1, L811.2
- new net: Q801.1 (G), R801.2, R802.1
- new net: R809.1, U812.8 (ICQ_ADJ)
- new net: RN802.3 (R3.1), RN802.4 (R4.1), U816.7 (CTRL)
- new net: RN802.1 (R1.1), RN802.2 (R2.1), U816.8 (EN)
- new net: RN801.1 (R1.1), RN801.2 (R2.1), U802.7 (CTRL)
- new net: RN801.3 (R3.1), RN801.4 (R4.1), U802.8 (EN)
- new net: R812.1, R813.2, U810.6 (Shut_Down)
- new net: R815.1, U811.3 (+), U813.3 (VOUT)
- new net: U803.2, U805.2 (IN)
- new net: C824.2, U813.5 (PCAP)
- new net 3V3: C801.1, U801.1 (IN)
- new net ANT: U816.2 (RF1)
- new net EN: R803.2, U801.3 (EN)
- new net FSENSE: R811.1, U811.9
- new net GNDA: C801.2, C805.1, C806.1, C809.2, C810.2, C811.1, C812.1, C815.2, C816.2, C818.2, C819.2, C820.2, C821.1, C822.1, C828.2, C829.2, R803.1, R804.1, R809.2, R813.1, R814.2, R815.2, R816.2, R817.2, R819.2, RN801.6 (R3.2), RN801.8 (R1.2), RN802.6 (R3.2), RN802.8 (R1.2), TP801.G, U801.2 (GND), U802.1 (GND), U802.10 (GND), U802.12 (GND), U802.13 (EP), U802.3 (GND), U802.4 (GND), U802.6 (GND), U803.3, U804.1 (GND), U804.2 (GND), U804.4 (GND), U804.5 (GND), U805.1 (GND), U805.3 (GND), U805.4 (GND), U805.5 (GND), U805.7 (GND), U805.8 (GND), U806.2 (GND), U808.1 (GND), U808.3 (GND), U808.4 (GND), U808.5 (GND), U808.7 (GND), U808.8 (GND), U810.1 (NIC), U810.3 (NIC), U810.4 (NIC), U810.5 (NIC), U810.8 (NIC), U810.9 (GND), U811.4 (VCC-), U812.1 (NIC), U812.4 (NIC), U812.9 (EP_GND), U813.2 (GND), U814.2 (GND), U815.1 (GND), U815.2 (GND), U815.3 (GND), U815.5 (GND), U815.6 (GND), U815.7 (GND), U816.1 (GND), U816.10 (GND), U816.12 (GND), U816.13 (EP), U816.3 (GND), U816.4 (GND), U816.6 (GND)
- new net PSENSE: R810.1, U811.1
- new net RFFE_3V3: C809.1, C810.1, C815.1, C818.1, C819.1, C820.1, C824.1, C826.2, L806.2, L810.2, Q801.2 (S), R801.1, RN801.5 (R4.2), RN802.7 (R2.2), U801.5 (OUT), U802.9 (VCC), U806.5 (VCC), U811.10 (VCC+), U812.5 (VCC), U813.4 (VCC), U814.4 (VCC), U816.9 (VCC)
- new net RFIO: U802.2 (RF1)
- new net RX_RF_IN: C817.2, U816.5 (RF3)
- new net RX_RF_OUT: U802.5 (RF3), U808.6 (OUT)
- new net TX_EN: R804.2, U806.1
- new net TX_RF_IN: U802.11 (RF2), U803.1
- new net TX_RF_OUT: TP801.A, U815.4 (OUT), U816.11 (RF2)
- new net ~{ΤX_EN}: R802.2, U806.3, U806.6
- new net ΤX_EN_ΙΝΤ: R808.2, R812.2, RN801.7 (R2.2), RN802.5 (R4.2), U806.4, U811.5 (EN1), U811.6 (EN2), U813.1 (~{SHDN}), U814.1 (~{SHDN})
- no-connect marks 0 -> 1
Other:
- note added: "+5.4dBm to + 26.0dBm"
- note added: "-10dBm to +15dBm"
- note added: "-23dBm to +2dBm"
- note added: "-9.1dBm to + 14.3dBm"
- note added: "RF1419D IL 1.6 dB Fc = 403.5 BW = 7.5 MHz This is placed after the 1st LNA to improve Detectivity"
- note added: "RF1419D This is placed before the HPA since it cannot handle the power Rated for 10dBm"
- note added: "RX Chain Power ON: TQP3M9036 -> 45mA Power STNDBY: TQP3M9036 -> 4mA Switching speeds: TQP3M9036 -> 1us Totals: ON state: < 45mA max OFF state: < 20uA Switch ON speed: 1 usec Switch OFF speed: 1 usec"
- note added: "TQP3M9036 NF = 0.45 Can be replaced by GRF2070 (NF=0.35) with small changes"
- note added: "TX Chain Power ON (no RF): 1x BGA6130 -> 71mA 1x QPA4263C-> 55mA 2x LTC5507 -> 1.7mA 2x TSV7723 -> 5mA Power ON (RF): 1x BGA6130 -> 200mA 1x QPA4263C-> 55mA 2x LTC5507 -> 1.7mA 2x TSV7723 -> 5mA Power STNDBY: 1x BGA6130 -> 6uA 1x QPA4263C-> 0mA 2x LTC5507 -> 8uA 2x TSV7723 -> 16uA Switching speeds: 1x BGA6130 -> 2.2us(PWRUP), 0.5us(PWRDN) 1x QPA4263C-> To be measured 2x LTC5507 -> 7-20us 2x TSV77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"
- note added: "The R divider ensures Ven<3V Making the board 5V compliant"
- note added: "The resistive tap is -25dB to ensure: * Dynamic range match to LTC5507 * Minimal power loss to main signal"
- note added: "This is needed to stop Tx_EN High during PWR_DN mode"

Commit message: implemented abstraction level page
Parts:
- removed C801, C809, C812: 1uF, Capacitor_SMD:C_0402_1005Metric, symbol Device:C
- removed C802, C804, C823, C824, C825, C826: 220pF, Capacitor_SMD:C_0402_1005Metric, symbol Device:C
- removed C803: 0 Ohm, Capacitor_SMD:C_0402_1005Metric, symbol Device:C
- removed C805, C808, C810, C817: 100pF, Capacitor_SMD:C_0402_1005Metric, symbol Device:C
- removed C806: 20pF, Capacitor_SMD:C_0402_1005Metric, symbol Device:C
- removed C807: 15pF, Capacitor_SMD:C_0402_1005Metric, symbol Device:C
- removed C811, C820, C827: 1nF, Capacitor_SMD:C_0402_1005Metric, symbol Device:C
- removed C815: 47nF, Capacitor_SMD:C_0402_1005Metric, symbol Device:C
- removed C816: 2.36pF, Capacitor_SMD:C_0402_1005Metric, symbol Device:C
- removed C818: 10uF, Capacitor_SMD:C_0402_1005Metric, symbol Device:C
- removed C819: 100nF, Capacitor_SMD:C_0402_1005Metric, symbol Device:C
- removed C821: Open, Capacitor_SMD:C_0402_1005Metric, symbol Device:C
- removed C822: 18pF, Capacitor_SMD:C_0402_1005Metric, symbol Device:C
- removed C828, C829: 10pF, Capacitor_SMD:C_0402_1005Metric, symbol Device:C
- removed L801, L806: 68nH, Inductor_SMD:L_0402_1005Metric, symbol Device:L
- removed L802: 18nH, Inductor_SMD:L_0402_1005Metric, symbol Device:L
- removed L809: 8.2nH, Inductor_SMD:L_0402_1005Metric, symbol Device:L
- removed L810: 68nH, Inductor_SMD:L_0603_1608Metric, symbol Device:L
- removed L811: 43 nH, Inductor_SMD:L_0402_1005Metric, symbol Device:L
- removed Q801: FDN308P, Package_TO_SOT_SMD:SOT-23, symbol Transistor_FET:FDN340P
- removed R801: 100k, Resistor_SMD:R_0402_1005Metric, symbol Device:R
- removed R802: 1k, Resistor_SMD:R_0402_1005Metric, symbol Device:R
- removed R803, R804, R810, R811, R813, R815, R817: 10k, Resistor_SMD:R_0402_1005Metric, symbol Device:R
- removed R805: 120, Resistor_SMD:R_0402_1005Metric, symbol Device:R
- removed R808: 270, Resistor_SMD:R_0402_1005Metric, symbol Device:R
- removed R809: 3k9, Resistor_SMD:R_0402_1005Metric, symbol Device:R
- removed R812: 33k, Resistor_SMD:R_0402_1005Metric, symbol Device:R
- removed R814, R816: 2k7, Resistor_SMD:R_0402_1005Metric, symbol Device:R
- removed R818: 453, Resistor_SMD:R_0402_1005Metric, symbol Device:R
- removed R819: 54.9, Resistor_SMD:R_0402_1005Metric, symbol Device:R
- removed RN801, RN802: 4.7k, Resistor_SMD:R_Array_Convex_4x0402, symbol Device:R_Pack04
- removed TP801: MS-156C3, lsf-kicad-lib:MS-156C3, symbol lsf-kicad:MS-156C3
- removed U801: BD226xG-M, lsf-kicad-lib:ROHM_SSOP-5, symbol lsf-kicad:BD226xG-M
- removed U802, U816: SKYA21003, lsf-kicad-lib:QFN-12-1EP_2x2mm_P0.5mm_EP0.76x0.76mm, symbol lsf-kicad:SKYA21003
- removed U803: PAT0816-C-10DB, lsf-kicad-lib:RF_Attenuator_Susumu_PAT0816, symbol RF:PAT1220-C-5DB
- removed U804: QPA4263C, Package_TO_SOT_SMD:SOT-363_SC-70-6, symbol lsf-kicad:QPA4263C
- removed U805, U808: RF1419D, lsf-kicad-lib:SM3838-8, symbol lsf-kicad:RF1419D
- removed U806: 74AUP2G14, Package_TO_SOT_SMD:SOT-363_SC-70-6, symbol lsf-kicad:74AUP2G14
- removed U810: TQP3M9036, lsf-kicad-lib:DFN-8-1EP_2x2mm_P0.5mm_EP0.7x1.6mm_ThermalVias, symbol lsf-kicad:TQP3M9036
- removed U811: TSV7723, Package_SO:MSOP-10_3x3mm_P0.5mm, symbol lsf-kicad:TSV7723
- removed U812: BGA6130, lsf-kicad-lib:NXP_HVSON-8, symbol lsf-kicad:BGA6130
- removed U813, U814: LTC5507ES6PBF, Package_TO_SOT_SMD:TSOT-23-6, symbol lsf-kicad:LTC5507
- removed U815: LFCG-490+, lsf-kicad-lib:GE0805C-2, symbol lsf-kicad:LFCG-490+
- added BOOT1: TD-1183SN-1.5H(3x2.5), NxtPX4:3x2.5PushButton, symbol Switch:SW_Push
- added C1, C12, C13, C3: 22uF(0805 35V 20%), Capacitor_SMD:C_0805_2012Metric, symbol Device:C_Small
- added C10, C16, C18, C19, C20, C33, C34, C37, C38, C39, C40, C43, C7: 100nF(0201 10V 10%), Capacitor_SMD:C_0201_0603Metric, symbol Device:C_Small
- added C11: 100nF(0201 16V 10%), Capacitor_SMD:C_0201_0603Metric, symbol Device:C_Small
- added C14, C15: 1uF(0402 10V 10%), Capacitor_SMD:C_0402_1005Metric, symbol Device:C_Small
- added C17, C21: 100nF(0201 25V 10%), Capacitor_SMD:C_0201_0603Metric, symbol Device:C_Small
- added C2: 10uF(0603 35V 20%), Capacitor_SMD:C_0603_1608Metric, symbol Device:C_Small
- added C22: 100nF(0201 10.0V 10%), Capacitor_SMD:C_0201_0603Metric, symbol Device:C_Small
- added C23, C24, C26: 22uF(0603 16V), Capacitor_SMD:C_0603_1608Metric, symbol Device:C_Small
- added C25: 10uF(0603 16V), Capacitor_SMD:C_0603_1608Metric, symbol Device:C_Small
- added C27, C28: 2.2uF(0402 6.3V 10%), Capacitor_SMD:C_0402_1005Metric, symbol Device:C_Small
- added C29: 4.7uF(0402 10V), Capacitor_SMD:C_0402_1005Metric, symbol Device:C_Small
- added C30: 15pF(0201 10V), Capacitor_SMD:C_0201_0603Metric, symbol Device:C_Small
- added C31: 100nF(0201 6.3V), Capacitor_SMD:C_0201_0603Metric, symbol Device:C_Small
- added C32: 1uF(0201 6.3V), Capacitor_SMD:C_0201_0603Metric, symbol Device:C_Small
- added C35, C36: 12.0pF(0201 10V), Capacitor_SMD:C_0201_0603Metric, symbol Device:C_Small
- added C4, C8: 1uF(0402 35V 10%), Capacitor_SMD:C_0402_1005Metric, symbol Device:C_Small
- added C41, C42, C44, C45: 100.0nF(0201 10V), Capacitor_SMD:C_0201_0603Metric, symbol Device:C_Small
- added C5, C6, C9: 1uF(0402 16V 10%), Capacitor_SMD:C_0402_1005Metric, symbol Device:C_Small
- added D1: PESD12VV1BL, NxtPX4:PESD12VV1BL_315, symbol Diode:ESD9B5.0ST5G
- added D10, D11, D8, D9: LED_Blue(0201), LED_SMD:LED_0201_0603Metric, symbol Device:LED_Small
- added D12: LED_RED(0201), LED_SMD:LED_0201_0603Metric, symbol Device:LED_Small
- added D13: LED_BLUE(0201), LED_SMD:LED_0201_0603Metric, symbol Device:LED_Small
- added D14: LED_Green(0201), LED_SMD:LED_0201_0603Metric, symbol Device:LED_Small
- added D2, D4: PESD5V0F1BL, NxtPX4:PESD5V0F1BL, symbol Diode:ESD9B5.0ST5G
- added D3: SMF30CA(30V), Diode_SMD:D_SOD-123F, symbol Device:D_TVS
- added D5, D7: DSS34(3A 500mV), Diode_SMD:D_SOD-123F, symbol Device:D_Schottky
- added D6: BZX584C9V1, Diode_SMD:D_SOD-523, symbol Device:D_Zener
- added FID1: Mark1, NxtPX4:Fidiucial, symbol Mechanical:Fiducial
- added FID2: Mark2, NxtPX4:Fidiucial, symbol Mechanical:Fiducial
- added FID3: Mark3, NxtPX4:Fidiucial, symbol Mechanical:Fiducial
- added H1, H2, H3, H4: MountingHole_Pad, NxtPX4:M2MountingHole, symbol Mechanical:MountingHole_Pad
- added J1: USB_C_Receptacle_USB2.0, NxtPX4:USB_C_Small, symbol Connector:USB_C_Receptacle_USB2.0
- added J10: Micro_SD_Card, NxtPX4:TF-SMD_TF-021B-H265, symbol Connector:Micro_SD_Card
- added J11: Debug, NxtPX4:1x06-1MP_P1.00mm_Horizontal, symbol Connector_Generic_MountingPin:Conn_01x06_MountingPin
- added J12: AuxGPIO, NxtPX4:1x06-1MP_P1.00mm_Horizontal, symbol Connector_Generic_MountingPin:Conn_01x06_MountingPin
- added J2: DJIO3, NxtPX4:1x06-1MP_P1.00mm_Horizontal, symbol Connector_Generic_MountingPin:Conn_01x06_MountingPin
- added J3: GPS, NxtPX4:1x06-1MP_P1.00mm_Horizontal, symbol Connector_Generic_MountingPin:Conn_01x06_MountingPin
- added J4: UART2, NxtPX4:01x04_MP_sh1.0_Hori, symbol Connector_Generic_MountingPin:Conn_01x04_MountingPin
- added J5, J7: Upper computer connector, NxtPX4:01x04_MP_sh1.0_Hori, symbol Connector_Generic_MountingPin:Conn_01x04_MountingPin
- added J6: ESC, NxtPX4:01x08_MP_sh1.0_Hori, symbol Connector_Generic_MountingPin:Conn_01x08_MountingPin
- added J8: PWM_AUX, NxtPX4:01x05_MP_sh1.0_Hori, symbol Connector_Generic_MountingPin:Conn_01x05_MountingPin
- added J9: Conn_01x04, NxtPX4:Conn_4Pin, symbol Connector_Generic:Conn_01x04
- added L1, L2: 10uH(0420)(78438357100), NxtPX4:Inductor_0420, symbol Device:L_Small
- added Q1: AP40P05, Package_TO_SOT_SMD:SOT-23, symbol Device:Q_PMOS_GSD
- added R1, R2: 5.1kR(0201), Resistor_SMD:R_0201_0603Metric, symbol Device:R_Small
- added R10, R8: 20R(0201 25V), Resistor_SMD:R_0201_0603Metric, symbol Device:R_Small
- added R11: 7.68kR(0201 25V), Resistor_SMD:R_0201_0603Metric, symbol Device:R_Small
- added R12, R9: 51kR(0201 25V), Resistor_SMD:R_0201_0603Metric, symbol Device:R_Small
- added R13, R17: 41.2kR(0201 25V), Resistor_SMD:R_0201_0603Metric, symbol Device:R_Small
- added R14: 200.0kR(0201 50V), Resistor_SMD:R_0201_0603Metric, symbol Device:R_Small
- added R15: 22.0kR(0201 50V), Resistor_SMD:R_0201_0603Metric, symbol Device:R_Small
- added R16: 2.90k-4.02kR(0201 25V) / 3k for 12V, Resistor_SMD:R_0201_0603Metric, symbol Device:R_Small
- added R18, R19, R20, R23, R27, R28, R31, R32, R33, R34, R35, R38: 10kR(0201), Resistor_SMD:R_0201_0603Metric, symbol Device:R_Small
- added R21: 20kR(0201 9V), Resistor_SMD:R_0201_0603Metric, symbol Device:R_Small
- added R24, R25, R26, R29, R30, R36, R37: 10.0kR(0201), Resistor_SMD:R_0201_0603Metric, symbol Device:R_Small
- added R3, R5: 1MR(0402 50V), Resistor_SMD:R_0402_1005Metric, symbol Device:R_Small
- added R4, R6: 100kR(0201 25V), Resistor_SMD:R_0201_0603Metric, symbol Device:R_Small
- added R7: 100kR(0201 50V), Resistor_SMD:R_0201_0603Metric, symbol Device:R_Small
- added TP1: 24V_TP, NxtPX4:MiniTP, symbol Connector:TestPoint
- added TP10, TP11, TP13, TP3, TP4, TP6, TP7, TP8: MP, NxtPX4:PWR_Circle, symbol Connector:TestPoint
- added TP12: CAM_9V, NxtPX4:MiniTP, symbol Connector:TestPoint
- added TP2: 3.3V_Core_TP, NxtPX4:MiniTP, symbol Connector:TestPoint
- added TP5: 3.3V_Peri_TP, NxtPX4:MiniTP, symbol Connector:TestPoint
- added TP9: 5V_System, NxtPX4:MiniTP, symbol Connector:TestPoint
- added U1, U4: MP9943GQ-Z, NxtPX4:MP9943GQ-Z, symbol NxtPX4_Symbol:MP9943GQ-Z
- added U10: Caution, NxtPX4:Caution, symbol NxtPX4_Symbol:Caution_Logo
- added U11: STM32H743VIH6, NxtPX4:STM32H743VIHBGA100C80P10X10_800X800X110N, symbol NxtPX4_Symbol:STM32H743VIH6
- added U13: SPL06, Package_LGA:Bosch_LGA-8_2x2.5mm_P0.65mm_ClockwisePinNumbering, symbol NxtPX4_Symbol:SPL06
- added U14, U15: BMI088, NxtPX4:BMI088, symbol NxtPX4_Symbol:BMI088
- added U16: W25Q128JVS, Package_SO:SOIC-8_5.23x5.23mm_P1.27mm, symbol Memory_Flash:W25Q128JVS
- added U17: UAV_LOGO, NxtPX4:Dual_logo, symbol NxtPX4_Symbol:Dual_Logo
- added U19: SN74LVC1G86DCKR, DCK5, symbol NxtPX4_Symbol:SN74LVC1G86DCKR
- added U2, U3: RT9013-33GB, NxtPX4:RT9013-33GB, symbol NxtPX4_Symbol:RT9013-33GB
- added U5: UAV_LOGO, NxtPX4:Uav_logo, symbol NxtPX4_Symbol:UAV_LOGO
- added U6: Direction_Logo, NxtPX4:Direction_Logo, symbol NxtPX4_Symbol:Direction_Logo
- added U8: Signature, NxtPX4:my_signature, symbol NxtPX4_Symbol:Signature
- added U9: high_voltage, NxtPX4:high_voltage, symbol NxtPX4_Symbol:High_Voltage_Logo
- added Y1: SG-210STF/ X1G004171002700, Oscillator:Oscillator_SMD_Abracon_ASDMB-4Pin_2.5x2.0mm, symbol NxtPX4_Symbol:SG-210STF
- added Y2: ABS07 (32.768kHZ), NxtPX4:LSE(2012), symbol NxtPX4_Symbol:LSE-Oscillator
Connections:
- new net: BOOT1.2, R28.2, U11.D5 (BOOT0)
- new net: R12.2, R16.2, R17.1
- new net: C7.1, R4.1, U1.2 (VCC)
- new net: R4.2, U1.8 (PG)
- new net: C21.1, R10.2
- new net: C21.2, L2.1, U4.6 (SW)
- new net: R3.2, U1.3 (EN/SYNC)
- new net: D12.1 (K), R24.1
- new net: D14.1 (K), R26.1
- new net: J1.A5 (CC1), R2.2
- new net: J1.B5 (CC2), R1.2
- new net: R12.1, U4.1 (FB)
- new net: C10.1, R6.1, U4.2 (VCC)
- new net: C30.1, U11.C1 (PH0-OSC_IN), Y1.3 (OUT)
- new net: D6.2 (A), Q1.1 (G), R7.1
- new net: C17.2, L1.1, U1.6 (SW)
- new net: D8.1 (K), R18.2
- new net: C35.1, U11.A1 (PC14-OSC32_IN), Y2.2
- new net: C36.1, U11.B1 (PC15-OSC32_OUT), Y2.1
- new net: C27.2, U11.E7 (VCAP)
- new net: C28.2, U11.F8 (VCAP)
- new net: R5.2, U4.3 (EN/SYNC)
- new net: R8.1, U1.4 (BST)
- new net: C17.1, R8.2
- new net: D10.1 (K), R20.2
- new net: D13.1 (K), R25.1
- new net: R11.2, R13.1, R9.2
- new net: R10.1, U4.4 (BST)
- new net: R6.2, U4.8 (PG)
- new net: R9.1, U1.1 (FB)
- new net: D9.1 (K), R19.2
- new net: D11.1 (K), R21.2
- new net ADC1_INP4_BATT_V: C22.1, R14.2, R15.1, U11.G4 (PC4)
- new net ADC2_INP8_BATT_I: J6.1 (Pin_1), U11.H4 (PC5)
- new net AUX1_PC0: J12.3 (Pin_3), U11.F1 (PC0)
- new net AUX2_PC1: J12.2 (Pin_2), U11.F2 (PC1)
- new net AUX3_PA4: J12.1 (Pin_1), U11.G3 (PA4)
- new net BMI088_0_ACS: U11.J2 (PA2), U15.14 (CSB1)
- new net BMI088_0_ADR: U11.G2 (PA0), U15.16 (INT1)
- new net BMI088_0_GCS: U11.K2 (PA3), U15.5 (CSB2)
- new net BMI088_0_GDR: U11.H2 (PA1), U15.12 (INT3)
- new net BMI088_0_MISO: U11.J3 (PA6), U15.10 (SDO2), U15.15 (SDO1)
- new net BMI088_0_MOSI: U11.K3 (PA7), U15.9 (SDI)
- new net BMI088_0_SCK: U11.H3 (PA5), U15.8 (SCK)
- new net BMI088_1_ACS: U11.A2 (PC13), U14.14 (CSB1)
- new net BMI088_1_ADR: U11.C3 (PE4), U14.16 (INT1)
- new net BMI088_1_GCS: U11.E2 (PC2_C), U14.5 (CSB2)
- new net BMI088_1_GDR: U11.B3 (PE3), U14.12 (INT3)
- new net BMI088_1_MISO: U11.D3 (PE5), U14.10 (SDO2), U14.15 (SDO1)
- new net BMI088_1_MOSI: U11.E3 (PE6), U14.9 (SDI)
- new net BMI088_1_SCK: U11.A3 (PE2), U14.8 (SCK)
- new net Baro_I2C1_DR: U11.C5 (PB5), U13.5 (SDO)
- new net Baro_I2C1_SCL: R36.1, U11.B5 (PB6), U13.4 (SCL)
- new net Baro_I2C1_SDA: R37.1, U11.A5 (PB7), U13.3 (SDA)
- new net CAM_9V: C25.1, C26.1, D11.2 (A), J2.1 (Pin_1), L2.2, R17.2, TP12.1
- new net Core_3V3: BOOT1.1, C14.1, C16.1, C19.1, C29.2, C31.1, C32.1, C34.1, C38.1, C40.1, C41.1, C42.1, C44.1, C45.1, D8.2 (A), R27.1, R29.2, R30.2, R31.2, R32.2, R33.2, R34.2, R35.2, R36.2, R37.2, TP2.1, U11.B2 (VBAT), U11.D2 (VDD), U11.D8 (PD0), U11.F4 (VDDLDO), U11.F5 (VDD), U11.F6 (VDD33USB), U11.F7 (PDR_ON), U11.H1 (VDDA), U11.K1 (VDD), U13.6 (VDDIO), U13.8 (VDD), U14.11 (VDDIO), U14.3 (VDD), U15.11 (VDDIO), U15.3 (VDD), U19.5 (VCC), U2.5 (VOUT), Y1.1 (~{ST}), Y1.4 (VCC)
- new net EX_I2C4_SCL: J3.5 (Pin_5), R29.1, U11.K10 (PD12)
- new net EX_I2C4_SDA: J3.6 (Pin_6), R30.1, U11.J10 (PD13)
- new net EX_SPI3_MISO: J12.5 (Pin_5), U11.A6 (PB4)
- new net EX_SPI3_MOSI: J12.4 (Pin_4), U11.G5 (PB2)
- new net EX_SPI3_SCK: J12.6 (Pin_6), U11.A7 (PB3)
- new net FRAM_SPI2_MISO: U11.H10 (PB14), U16.2 (DO(IO1))
- new net FRAM_SPI2_MOSI: U11.F3 (PC3_C), U16.5 (DI(IO0))
- new net FRAM_SPI2_SCK: U11.C7 (PD3), U16.6 (CLK)
- new net FRAM_SPI2_~{CS}: U11.D7 (PD4), U16.1 (~{CS})
- new net GND: C1.2, C10.2, C11.2, C12.2, C13.2, C14.2, C15.2, C16.2, C18.2, C19.2, C2.2, C20.2, C22.2, C23.2, C24.2, C25.2, C26.2, C27.1, C28.1, C29.1, C3.2, C30.2, C31.2, C32.2, C33.2, C34.2, C35.2, C36.2, C37.2, C38.2, C39.2, C4.2, C40.2, C41.2, C42.2, C43.1, C44.2, C45.2, C5.2, C6.2, C7.2, C8.2, C9.2, D1.1 (A1), D2.1 (A1), D3.1 (A1), D4.1 (A1), H1.1, H2.1, H3.1, H4.1, J1.A1 (GND), J1.A12 (GND), J1.B1 (GND), J1.B12 (GND), J1.S1 (SHIELD), J10.6 (VSS), J10.9 (SHIELD), J11.1 (Pin_1), J11.MP (MountPin), J12.MP (MountPin), J2.2 (Pin_2), J2.5 (Pin_5), J2.MP (MountPin), J3.1 (Pin_1), J3.MP (MountPin), J4.1 (Pin_1), J4.MP (MountPin), J5.1 (Pin_1), J5.MP (MountPin), J6.8 (Pin_8), J6.MP (MountPin), J7.1 (Pin_1), J7.MP (MountPin), J8.1 (Pin_1), J8.MP (MountPin), J9.4 (Pin_4), R1.1, R11.1, R15.2, R16.1, R18.1, R19.1, R2.1, R20.1, R21.1, R23.1, R24.2, R25.2, R26.2, R28.1, R38.1, R7.2, TP10.1, TP11.1, TP13.1, TP8.1, U1.5 (GND), U11.C2 (VSS), U11.E4 (VSS), U11.E5 (VSS), U11.E6 (VSS), U11.G1 (VSSA), U11.J1 (VSS), U13.1 (GND), U13.7 (GND), U14.4 (GNDIO), U14.6 (GND), U14.7 (PS), U15.4 (GNDIO), U15.6 (GND), U15.7 (PS), U16.4 (GND), U19.3 (GND), U2.2 (GND), U3.2 (GND), U4.5 (GND), Y1.2 (GND)
- new net LED_BLUE: D13.2 (A), U11.G10 (PB15)
- new net LED_GREEN: D14.2 (A), U11.G9 (PD11)
- new net LED_RED: D12.2 (A), U11.G8 (PD15)
- new net NRST: C33.1, R27.2, U11.E1 (NRST)
- new net Periph_3V3: C15.1, C18.1, C20.1, C37.1, C39.1, C43.2, D9.2 (A), J10.4 (VDD), TP5.1, U16.3 (IO2), U16.7 (IO3), U16.8 (VCC), U3.5 (VOUT)
- new net SBUS: J2.6 (Pin_6), J7.4 (Pin_4), R23.2, U19.2
- new net SBUS_INV: R38.2, U11.H8 (PD14), U19.1
- new net SCLK: J11.5 (Pin_5), U11.A9 (PA14)
- new net SDMMC1_CK: J10.5 (CLK), U11.C8 (PC12)
- new net SDMMC1_CMD: J10.3 (CMD), R33.1, U11.B7 (PD2)
- new net SDMMC1_D0: J10.7 (DAT0), R34.1, U11.F9 (PC8)
- new net SDMMC1_D1: J10.8 (DAT1), R35.1, U11.E9 (PC9)
- new net SDMMC1_D2: J10.1 (DAT2), R31.1, U11.B9 (PC10)
- new net SDMMC1_D3: J10.2 (DAT3/CD), R32.1, U11.B8 (PC11)
- new net SWDIO: J11.6 (Pin_6), U11.A10 (PA13)
- new net System_4V5: C5.1, C6.1, D5.1 (K), D7.1 (K), U2.1 (VIN), U2.3 (EN), U3.1 (VIN), U3.3 (EN)
- new net System_5V: C23.1, C24.1, D10.2 (A), D7.2 (A), J11.2 (Pin_2), J3.2 (Pin_2), J4.2 (Pin_2), J5.2 (Pin_2), J7.2 (Pin_2), L1.2, R13.2, TP3.1, TP4.1, TP6.1, TP7.1, TP9.1
- new net TIM1_CH1: J6.3 (Pin_3), U11.K5 (PE9)
- new net TIM1_CH2: J6.4 (Pin_4), U11.H6 (PE11)
- new net TIM1_CH3: J6.5 (Pin_5), U11.K6 (PE13)
- new net TIM1_CH4: J6.6 (Pin_6), U11.G7 (PE14)
- new net TIM2_CH3: J8.4 (Pin_4), U11.J7 (PB10)
- new net TIM2_CH4: J8.5 (Pin_5), U11.K7 (PB11)
- new net TIM3_CH3: J8.3 (Pin_3), U11.J4 (PB0)
- new net TIM3_CH4: J8.2 (Pin_2), U11.K4 (PB1)
- new net UART4_RX: J5.4 (Pin_4), U11.B4 (PB8)
- new net UART4_TX: J5.3 (Pin_3), U11.A4 (PB9)
- new net UART5_RX: U11.K8 (PB12), U19.4
- new net UART5_TX: J7.3 (Pin_3), U11.J8 (PB13)
- new net UART6_RX: U11.E10 (PC7)
- new net UART6_TX: U11.F10 (PC6)
- new net UART7_RX: J6.2 (Pin_2), U11.H5 (PE7)
- new net UART7_TX: U11.J5 (PE8)
- new net UART8_RX: J11.4 (Pin_4), U11.D4 (PE0)
- new net UART8_TX: J11.3 (Pin_3), U11.C4 (PE1)
- new net USART1_CK: U11.D9 (PA8)
- new net USART1_RX: J3.4 (Pin_4), U11.D10 (PA10)
- new net USART1_TX: J3.3 (Pin_3), U11.C9 (PA9)
- new net USART2_CK: U11.D6 (PD7)
- new net USART2_RX: J4.4 (Pin_4), U11.C6 (PD6)
- new net USART2_TX: J4.3 (Pin_3), U11.B6 (PD5)
- new net USART3_CK: U11.H9 (PD10)
- new net USART3_RX: J2.4 (Pin_4), U11.J9 (PD9)
- new net USART3_TX: J2.3 (Pin_3), U11.K9 (PD8)
- new net USB_OTG_FS_DM: D2.2 (A2), J1.A7 (D-), J1.B7 (D-), J9.2 (Pin_2), U11.C10 (PA11)
- new net USB_OTG_FS_DP: D4.2 (A2), J1.A6 (D+), J1.B6 (D+), J9.3 (Pin_3), U11.B10 (PA12)
- new net VBUS: C11.1, C9.1, D1.2 (A2), D5.2 (A), J1.A4 (VBUS), J1.A9 (VBUS), J1.B4 (VBUS), J1.B9 (VBUS), J9.1 (Pin_1)
- new net VCC_24V: C1.1, C2.1, C3.1, C4.1, C8.1, D6.1 (K), Q1.2 (S), R14.1, R3.1, R5.1, TP1.1, U1.7 (IN), U4.7 (IN)
- new net VCC_BAT: C12.1, C13.1, D3.2 (A2), J6.7 (Pin_7), Q1.3 (D)
- no-connect marks 1 -> 19
Other:
- note added: "2S-6S input to 5V"
- note added: "2S-6S input to 9V"
- note added: "3.3V 500mA MCU IMU Power"
- note added: "3.3V 500mA TF-Card QSPI OSD"
- note added: "3.54k output 10V 4.02k output 9V 2.9k for 12V"
- note added: "5V 3A output"
- note added: "5V to Core_VCC"
- note added: "5V to Periph_VCC"
- note added: "7.68kR 5V output"
- note added: "9V 3A output"
- note added: "9V/10V to drive CAM"
- note added: "ADR for accel data ready GDR for gyro data ready ACS for accel cs GCS for gyro cs"
- note added: "BAT power"
- note added: "BAT power protection"
- note added: "BAT_Voltage_Detection"
- note added: "Buzzer"
- note added: "Cap should be 10% X5R Res should be 1%"
- note added: "DJI O3"
- note added: "FRAM / QSPI"
- note added: "IMU BMI088 SPI1"
- note added: "IMU BMI088 SPI4"
- note added: "IO GH2.5"
- note added: "If 0R is connected UART5 RX is used as SBUS"
- note added: "If want to utilize UART8 in PX4, make UART6 as the debug port"
- note added: "MCU"
- note added: "SDO To VSS ADDR:0x1110110 SDO To VDDIO ADDR:0x1110111 CSB To VDDIO In I2C Mode"
- note added: "SD_CARD"
- note added: "SPL06 Baro I2C1"
- note added: "Sbus"
- note added: "Type-C power"
- note added: "power up singal to tirgger qgroundcontrol bootloader sync"
- note removed: "+5.4dBm to + 26.0dBm"
- note removed: "-10dBm to +15dBm"
- note removed: "-23dBm to +2dBm"
- note removed: "-9.1dBm to + 14.3dBm"
- note removed: "RF1419D IL 1.6 dB Fc = 403.5 BW = 7.5 MHz This is placed after the 1st LNA to improve Detectivity"
- note removed: "RF1419D This is placed before the HPA since it cannot handle the power Rated for 10dBm"
- note removed: "RX Chain Power ON: TQP3M9036 -> 45mA Power STNDBY: TQP3M9036 -> 4mA Switching speeds: TQP3M9036 -> 1us Totals: ON state: < 45mA max OFF state: < 20uA Switch ON speed: 1 usec Switch OFF speed: 1 usec"
- note removed: "TQP3M9036 NF = 0.45 Can be replaced by GRF2070 (NF=0.35) with small changes"
- note removed: "TX Chain Power ON (no RF): 1x BGA6130 -> 71mA 1x QPA4263C-> 55mA 2x LTC5507 -> 1.7mA 2x TSV7723 -> 5mA Power ON (RF): 1x BGA6130 -> 200mA 1x QPA4263C-> 55mA 2x LTC5507 -> 1.7mA 2x TSV7723 -> 5mA Power STNDBY: 1x BGA6130 -> 6uA 1x QPA4263C-> 0mA 2x LTC5507 -> 8uA 2x TSV7723 -> 16uA Switching speeds: 1x BGA6130 -> 2.2us(PWRUP), 0.5us(PWRDN) 1x QPA4263C-> To be measured 2x LTC5507 -> 7-20us 2x TSV77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"
- note removed: "The R divider ensures Ven<3V Making the board 5V compliant"
- note removed: "The resistive tap is -25dB to ensure: * Dynamic range match to LTC5507 * Minimal power loss to main signal"
- note removed: "This is needed to stop Tx_EN High during PWR_DN mode"
- company: (none) -> HKUST Khalil
- title: (none) -> NxtPX4
